File: Endstufe.kicad_sch (KiCad schematic)
At the start: 4 parts

Commit message: Completed first design
Parts:
- added H5, H6: MountingHole, Endstufe:MountingHole_3.2mm_M3_ISO14580_Pad, symbol Endstufe:MountingHole_Pad
- H1, H2, H3, H4: footprint footprints:MountingHole_3.2mm_M3_ISO14580_Pad -> Endstufe:MountingHole_3.2mm_M3_ISO14580_Pad
Connections:
- net GND: now also H5.1, H6.1
Changed lines of the file:
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@@
     (effects (font (size 1.27 1.27)) (justify left bottom))
+  )
+  (symbol (lib_id "Endstufe:MountingHole_Pad") (at 33.02 175.26 90) (unit 1)
+    (in_bom yes) (on_board yes) (dnp no) (fields_autoplaced)
+    (property "Reference" "H6" (at 29.21 176.53 90)
+      (effects (font (size 1.27 1.27)) (justify left))
+    )
+    (property "Value" "MountingHole" (at 29.21 173.99 90)
+      (effects (font (size 1.27 1.27)) (justify left))
+    )
+    (property "Footprint" "Endstufe:MountingHole_3.2mm_M3_ISO14580_Pad" (at 33.02 175.26 0)
+      (effects (font (size 1.27 1.27)) hide)
+    )
+    (property "Datasheet" "~" (at 33.02 175.26 0)
+      (effects (font (size 1.27 1.27)) hide)
+    )
+    (pin "1")
+    (instances
+      (project "Endstufe"
+        (path "/204ecd4a-024c-4bd2-9ce8-9773ce5b0d88"
+          (reference "H6") (unit 1)
+        )
+      )
+    )
   )
   (symbol (lib_id "Endstufe:MountingHole_Pad") (at 38.1 175.26 270) (unit 1)
@@
       (effects (font (size 1.27 1.27)) (justify left))
     )
-    (property "Footprint" "footprints:MountingHole_3.2mm_M3_ISO14580_Pad" (at 38.1 175.26 0)
+    (property "Footprint" "Endstufe:MountingHole_3.2mm_M3_ISO14580_Pad" (at 38.1 175.26 0)
       (effects (font (size 1.27 1.27)) hide)
     )
@@
       (effects (font (size 1.27 1.27)) (justify left))
     )
-    (property "Footprint" "footprints:MountingHole_3.2mm_M3_ISO14580_Pad" (at 38.1 165.1 0)
+    (property "Footprint" "Endstufe:MountingHole_3.2mm_M3_ISO14580_Pad" (at 38.1 165.1 0)
       (effects (font (size 1.27 1.27)) hide)
     )
@@
     )
   )
+  (symbol (lib_id "Endstufe:MountingHole_Pad") (at 33.02 180.34 90) (unit 1)
+    (in_bom yes) (on_board yes) (dnp no) (fields_autoplaced)
+    (property "Reference" "H5" (at 29.21 181.61 90)
+      (effects (font (size 1.27 1.27)) (justify left))
+    )
+    (property "Value" "MountingHole" (at 29.21 179.07 90)
+      (effects (font (size 1.27 1.27)) (justify left))
+    )
+    (property "Footprint" "Endstufe:MountingHole_3.2mm_M3_ISO14580_Pad" (at 33.02 180.34 0)
+      (effects (font (size 1.27 1.27)) hide)
+    )
+    (property "Datasheet" "~" (at 33.02 180.34 0)
+      (effects (font (size 1.27 1.27)) hide)
+    )
+    (pin "1")
+    (instances
+      (project "Endstufe"
+        (path "/204ecd4a-024c-4bd2-9ce8-9773ce5b0d88"
+          (reference "H5") (unit 1)
+        )
+      )
+    )
+  )
   (symbol (lib_id "Endstufe:MountingHole_Pad") (at 38.1 170.18 270) (unit 1)
     (in_bom yes) (on_board yes) (dnp no) (fields_autoplaced)
@@
       (effects (font (size 1.27 1.27)) (justify left))
     )
-    (property "Footprint" "footprints:MountingHole_3.2mm_M3_ISO14580_Pad" (at 38.1 170.18 0)
+    (property "Footprint" "Endstufe:MountingHole_3.2mm_M3_ISO14580_Pad" (at 38.1 170.18 0)
       (effects (font (size 1.27 1.27)) hide)
     )
@@
       (effects (font (size 1.27 1.27)) (justify left))
     )
-    (property "Footprint" "footprints:MountingHole_3.2mm_M3_ISO14580_Pad" (at 38.1 180.34 0)
+    (property "Footprint" "Endstufe:MountingHole_3.2mm_M3_ISO14580_Pad" (at 38.1 180.34 0)
       (effects (font (size 1.27 1.27)) hide)
     )
