File: RP2040.kicad_sch (KiCad schematic)
At the start: 34 parts, among them J22 DNP, J23 DNP, J24 DNP, J27 DNP, J28 DNP, J30 DNP, SW1 TS-1187A-B-A-B, SW2 TS-1187A-B-A-B, U10 TYPE-C 16PFS 2JCB1.2-H6.5 IPX8, U8 RP2040, U9 W25Q128JVS, Y3 12Mhz

Commit message: Completed first design
Connections:
- net +24V: now also J24.5 (Pin_5)
- net GND: no longer J24.5 (Pin_5)
Changed lines of the file:
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@@
   (junction (at 252.73 66.04) (diameter 0) (color 0 0 0 0)
   )
-  (junction (at 125.73 180.34) (diameter 0) (color 0 0 0 0)
-  )
   (junction (at 191.77 36.83) (diameter 0) (color 0 0 0 0)
   )
@@
   )
   (junction (at 148.59 63.5) (diameter 0) (color 0 0 0 0)
+  )
+  (junction (at 138.43 172.72) (diameter 0) (color 0 0 0 0)
   )
   (junction (at 204.47 29.21) (diameter 0) (color 0 0 0 0)
@@
     (stroke (width 0) (type default))
   )
-  (wire (pts (xy 138.43 180.34) (xy 125.73 180.34))
-    (stroke (width 0) (type default))
-  )
   (wire (pts (xy 162.56 137.16) (xy 162.56 124.46))
     (stroke (width 0) (type default))
@@
     (stroke (width 0) (type default))
   )
-  (wire (pts (xy 138.43 175.26) (xy 138.43 180.34))
-    (stroke (width 0) (type default))
-  )
   (wire (pts (xy 240.03 127) (xy 246.38 127))
     (stroke (width 0) (type default))
@@
     (stroke (width 0) (type default))
   )
+  (wire (pts (xy 138.43 172.72) (xy 138.43 175.26))
+    (stroke (width 0) (type default))
+  )
