File: Endstufe_v2/ControlBoard/DAC_Filter.kicad_sch (KiCad schematic)
At the start: 7 parts

Commit message: Change unavailable parts to available ones, optimise silkscreen, do via stiching
Parts:
- C95: footprint Capacitor_SMD:C_0402_1005Metric -> Endstufe:C_0402_1005Metric
Changed lines of the file:
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@@
 			)
 		)
-		(property "Footprint" "Capacitor_SMD:C_0402_1005Metric"
+		(property "Footprint" "Endstufe:C_0402_1005Metric"
 			(at 132.588 93.98 90)
 			(effects
