File: Endstufe_v2/ControlBoard/Power.kicad_sch (KiCad schematic)
At the start: 21 parts, among them J17 Conn_01x02_Pin, J18 Conn_01x02_Pin, J6 Conn_01x02_Pin, J7 DNP, U1 NVTFWS014P04M8LTAG, U2 1SMA5927A, U3 TPS62933

Commit message: Change unavailable parts to available ones, optimise silkscreen, do via stiching
Parts:
- J17, J18, J6: footprint Connector_JST:JST_XH_B2B-XH-A_1x02_P2.50mm_Vertical -> Endstufe:JST_XH_B2B-XH-A_1x02_P2.50mm_Vertical; JLCPCB Position Offset (none) -> 0,-0.5; LCSC (none) -> C158012
- L1: footprint Endstufe:L2520 -> Endstufe:IND-SMD_L4.4-W4.2; LCSC Part # C280577 -> C167206
- TP1: footprint TestPoint:TestPoint_Pad_D1.0mm -> Endstufe:TestPoint_Pad_D1.0mm
- U3: LCSC Part # C3200405 -> C6290372
Changed lines of the file:
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@@
 			)
 		)
-		(property "Footprint" "Connector_JST:JST_XH_B2B-XH-A_1x02_P2.50mm_Vertical"
+		(property "Footprint" "Endstufe:JST_XH_B2B-XH-A_1x02_P2.50mm_Vertical"
 			(at 214.63 147.32 0)
 			(effects
@@
 			)
 		)
+		(property "JLCPCB Position Offset" "0,-0.5"
+			(at 0 294.64 0)
+			(effects
+				(font
+					(size 1.27 1.27)
+				)
+				(hide yes)
+			)
+		)
+		(property "LCSC" "C158012"
+			(at 0 294.64 0)
+			(effects
+				(font
+					(size 1.27 1.27)
+				)
+				(hide yes)
+			)
+		)
 		(pin "1"
 		)
@@
 			)
 		)
-		(property "Footprint" "Connector_JST:JST_XH_B2B-XH-A_1x02_P2.50mm_Vertical"
+		(property "Footprint" "Endstufe:JST_XH_B2B-XH-A_1x02_P2.50mm_Vertical"
 			(at 214.63 134.62 0)
 			(effects
@@
 			)
 		)
+		(property "JLCPCB Position Offset" "0,-0.5"
+			(at 0 269.24 0)
+			(effects
+				(font
+					(size 1.27 1.27)
+				)
+				(hide yes)
+			)
+		)
+		(property "LCSC" "C158012"
+			(at 0 269.24 0)
+			(effects
+				(font
+					(size 1.27 1.27)
+				)
+				(hide yes)
+			)
+		)
 		(pin "1"
 		)
@@
 			)
 		)
-		(property "Footprint" "Connector_JST:JST_XH_B2B-XH-A_1x02_P2.50mm_Vertical"
+		(property "Footprint" "Endstufe:JST_XH_B2B-XH-A_1x02_P2.50mm_Vertical"
 			(at 83.82 152.4 0)
 			(effects
@@
 			)
 		)
+		(property "JLCPCB Position Offset" "0,-0.5"
+			(at 0 304.8 0)
+			(effects
+				(font
+					(size 1.27 1.27)
+				)
+				(hide yes)
+			)
+		)
+		(property "LCSC" "C158012"
+			(at 0 304.8 0)
+			(effects
+				(font
+					(size 1.27 1.27)
+				)
+				(hide yes)
+			)
+		)
 		(pin "1"
 		)
@@
 			)
 		)
-		(property "Footprint" "TestPoint:TestPoint_Pad_D1.0mm"
+		(property "Footprint" "Endstufe:TestPoint_Pad_D1.0mm"
 			(at 135.89 66.04 0)
 			(effects
@@
 			)
 		)
-		(property "Footprint" "Endstufe:L2520"
+		(property "Footprint" "Endstufe:IND-SMD_L4.4-W4.2"
 			(at 186.69 76.2 0)
 			(effects
@@
 			)
 		)
-		(property "LCSC Part #" "C280577"
+		(property "LCSC Part #" "C167206"
 			(at 186.69 76.2 0)
 			(effects
@@
 			)
 		)
-		(property "LCSC Part #" "C3200405"
+		(property "LCSC Part #" "C6290372"
 			(at 143.51 76.2 0)
 			(effects
