File: Endstufe_v2/InputBoard/PCM1865.kicad_sch (KiCad schematic)
At the start: 21 parts, among them J1 ST-0322D00-071-1A2H, J2 ST-0322D00-071-1A2H, J3 ST-0322D00-071-1A2H, J4 ST-0322D00-071-1A2H, U1 PCM1865DBTR, Y1 24.576Mhz

Commit message: Change unavailable parts to available ones, optimise silkscreen, do via stiching
Parts:
- C5, C6: LCSC Part # C458861 -> C526980
- J1, J2, J3, J4: JLCPCB Position Offset (none) -> 1.5,-0.1
- U1: JLCPCB Rotation Offset (none) -> 90
Changed lines of the file:
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@@
+			)
+		)
+		(property "JLCPCB Position Offset" "1.5,-0.1"
+			(at 0 139.7 0)
+			(effects
+				(font
+					(size 1.27 1.27)
+				)
+				(hide yes)
 			)
 		)
@@
 			)
 		)
+		(property "JLCPCB Rotation Offset" "90"
+			(at 0 205.74 0)
+			(effects
+				(font
+					(size 1.27 1.27)
+				)
+				(hide yes)
+			)
+		)
 		(pin "1"
 		)
@@
 			)
 		)
+		(property "JLCPCB Position Offset" "1.5,-0.1"
+			(at 0 53.34 0)
+			(effects
+				(font
+					(size 1.27 1.27)
+				)
+				(hide yes)
+			)
+		)
 		(pin "1"
 		)
@@
 			)
 		)
-		(property "LCSC Part #" "C458861"
+		(property "LCSC Part #" "C526980"
 			(at 137.16 114.3 0)
 			(effects
@@
 			)
 		)
-		(property "LCSC Part #" "C458861"
+		(property "LCSC Part #" "C526980"
 			(at 137.16 129.54 0)
 			(effects
@@
 			)
 		)
+		(property "JLCPCB Position Offset" "1.5,-0.1"
+			(at 0 228.6 0)
+			(effects
+				(font
+					(size 1.27 1.27)
+				)
+				(hide yes)
+			)
+		)
 		(pin "1"
 		)
@@
 			(effects
 				(font
+					(size 1.27 1.27)
+				)
+				(hide yes)
+			)
+		)
+		(property "JLCPCB Position Offset" "1.5,-0.1"
+			(at 0 314.96 0)
+			(effects
+				(font
