File: Endstufe_v2/InputBoard/PCM9211.kicad_sch (KiCad schematic)
At the start: 25 parts, among them U2 PCM9211PTR, U4 ZPLR135_T8, U5 ZPLR135_T8, U6 ZPLR135_T8, U7 ZPLR135_T8, Y2 24.576Mhz

Commit message: Change unavailable parts to available ones, optimise silkscreen, do via stiching
Parts:
- C12, C13: LCSC Part # C458861 -> C526980
- C21: LCSC Part # C361177 -> C77084
- R4: LCSC Part # C852886 -> C2684537
- U2: JLCPCB Rotation Offset (none) -> 90
- U4, U5, U6, U7: footprint CONN-TH_ZPLR135-T8 -> Endstufe:CONN-TH_ZPLR135-T8; JLCPCB Position Offset (none) -> 0,-3
Changed lines of the file:
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@@
 			)
 		)
-		(property "Footprint" "CONN-TH_ZPLR135-T8"
+		(property "Footprint" "Endstufe:CONN-TH_ZPLR135-T8"
 			(at 44.45 41.91 0)
 			(effects
@@
 		(property "LCSC" "C277778"
 			(at 44.45 31.75 0)
+			(effects
+				(font
+					(size 1.27 1.27)
+				)
+				(hide yes)
+			)
+		)
+		(property "JLCPCB Position Offset" "0,-3"
+			(at 0 63.5 0)
 			(effects
 				(font
@@
 			)
 		)
-		(property "LCSC Part #" "C458861"
+		(property "LCSC Part #" "C526980"
 			(at 33.02 101.6 0)
 			(effects
@@
 			)
 		)
-		(property "Footprint" "CONN-TH_ZPLR135-T8"
+		(property "Footprint" "Endstufe:CONN-TH_ZPLR135-T8"
 			(at 80.01 41.91 0)
 			(effects
@@
 		(property "LCSC" "C277778"
 			(at 80.01 31.75 0)
+			(effects
+				(font
+					(size 1.27 1.27)
+				)
+				(hide yes)
+			)
+		)
+		(property "JLCPCB Position Offset" "0,-3"
+			(at 0 63.5 0)
 			(effects
 				(font
@@
 			)
 		)
+		(property "JLCPCB Rotation Offset" "90"
+			(at 0 76.2 0)
+			(effects
+				(font
+					(size 1.27 1.27)
+				)
+				(hide yes)
+			)
+		)
 		(pin "1"
 		)
@@
 			)
 		)
+		(property "JLCPCB Rotation Offset" "90"
+			(at 0 157.48 0)
+			(effects
+				(font
+					(size 1.27 1.27)
+				)
+				(hide yes)
+			)
+		)
 		(pin "1"
 		)
@@
 			)
 		)
-		(property "Footprint" "CONN-TH_ZPLR135-T8"
+		(property "Footprint" "Endstufe:CONN-TH_ZPLR135-T8"
 			(at 151.13 41.91 0)
 			(effects
@@
 		(property "LCSC" "C277778"
 			(at 151.13 31.75 0)
+			(effects
+				(font
+					(size 1.27 1.27)
+				)
+				(hide yes)
+			)
+		)
+		(property "JLCPCB Position Offset" "0,-3"
+			(at 0 63.5 0)
 			(effects
 				(font
@@
 			)
 		)
-		(property "LCSC Part #" "C852886"
+		(property "LCSC Part #" "C2684537"
 			(at 271.78 52.07 0)
 			(effects
@@
 			)
 		)
-		(property "Footprint" "CONN-TH_ZPLR135-T8"
+		(property "Footprint" "Endstufe:CONN-TH_ZPLR135-T8"
 			(at 115.57 41.91 0)
 			(effects
@@
 		(property "LCSC" "C277778"
 			(at 115.57 31.75 0)
+			(effects
+				(font
+					(size 1.27 1.27)
+				)
+				(hide yes)
+			)
+		)
+		(property "JLCPCB Position Offset" "0,-3"
+			(at 0 63.5 0)
 			(effects
 				(font
@@
 			)
 		)
-		(property "LCSC Part #" "C361177"
+		(property "LCSC Part #" "C77084"
 			(at 271.78 44.45 0)
 			(effects
@@
 			)
 		)
-		(property "LCSC Part #" "C458861"
+		(property "LCSC Part #" "C526980"
 			(at 33.02 116.84 0)
 			(effects
